Commit message: Added joint space planning with Gazebo Simulation

File: src/robot_arm_model/urdf/robot_arm_model.urdf.xacro (robot description, xacro)
@@ -2,4 +2,8 @@
 <robot
   name="robot_arm_model" xmlns:xacro="http://www.ros.org/wiki/xacro">
+  <!-- Macros -->
+  <!-- <xacro:include filename="$(find robot_arm_model)/urdf/arm_base_gazebo.xacro" /> -->
+  <xacro:include filename="$(find robot_arm_model)/urdf/arm_model_control.xacro" />
+  <!-- Robot Model -->
   <link
     name="base_link">
@@ -29,5 +33,5 @@
         name="">
         <color
-          rgba="0.792156862745098 0.819607843137255 0.933333333333333 1" />
+          rgba="0.1 0.1 0.1 1" />
       </material>
     </visual>
@@ -69,5 +73,5 @@
         name="">
         <color
-          rgba="0.792156862745098 0.819607843137255 0.933333333333333 1" />
+          rgba="1.0 0.0 0.0 1" />
       </material>
     </visual>
@@ -97,6 +101,6 @@
       lower="-3.14"
       upper="3.14"
-      effort="0"
-      velocity="0" />
+      effort="3"
+      velocity="4.5" />
   </joint>
   <link
@@ -127,5 +131,5 @@
         name="">
         <color
-          rgba="0.792156862745098 0.819607843137255 0.933333333333333 1" />
+          rgba="0.1 0.1 0.1 1" />
       </material>
     </visual>
@@ -155,6 +159,6 @@
       lower="-1.57"
       upper="1.57"
-      effort="0"
-      velocity="0" />
+      effort="3"
+      velocity="4.5" />
   </joint>
   <link
@@ -185,5 +189,5 @@
         name="">
         <color
-          rgba="0.792156862745098 0.819607843137255 0.933333333333333 1" />
+          rgba="0.0 0.0 1.0 1" />
       </material>
     </visual>
@@ -213,6 +217,6 @@
       lower="-3.14"
       upper="3.14"
-      effort="0"
-      velocity="0" />
+      effort="3"
+      velocity="4.5" />
   </joint>
   <link
@@ -243,5 +247,5 @@
         name="">
         <color
-          rgba="0.792156862745098 0.819607843137255 0.933333333333333 1" />
+          rgba="0.1 0.1 0.1 1" />
       </material>
     </visual>
@@ -271,6 +275,6 @@
       lower="-3.14"
       upper="3.14"
-      effort="0"
-      velocity="0" />
+      effort="3"
+      velocity="4.5" />
   </joint>
   <link
@@ -301,5 +305,5 @@
         name="">
         <color
-          rgba="0.792156862745098 0.819607843137255 0.933333333333333 1" />
+          rgba="0.1 0.1 0.1 1" />
       </material>
     </visual>
@@ -329,6 +333,6 @@
       lower="-1.57"
       upper="1.57"
-      effort="0"
-      velocity="0" />
+      effort="3"
+      velocity="4.5" />
   </joint>
   <link
@@ -385,3 +389,43 @@
       xyz="1 0 0" />
   </joint>
+  <ros2_control name="5DofPosition" type="system">
+    <hardware>
+      <plugin>gz_ros2_control/GazeboSimSystem</plugin>
+    </hardware>
+    <joint name="Joint_1">
+      <command_interface name="position"/>
+      <state_interface name="position">
+        <param name="initial_value">0.0</param>
+      </state_interface>
+      <state_interface name="velocity"/>
+    </joint>
+    <joint name="Joint_2">
+      <command_interface name="position"/>
+      <state_interface name="position">
+        <param name="initial_value">0.0</param>
+      </state_interface>
+      <state_interface name="velocity"/>
+      </joint>
+      <joint name="Joint_3">
+        <command_interface name="position"/>
+        <state_interface name="position">
+          <param name="initial_value">0.0</param>
+        </state_interface>
+        <state_interface name="velocity"/>
+      </joint>
+      <joint name="Joint_4">
+        <command_interface name="position"/>
+        <state_interface name="position">
+          <param name="initial_value">0.0</param>
+        </state_interface>
+        <state_interface name="velocity"/>
+      </joint>
+      <joint name="Joint_5">
+        <command_interface name="position"/>
+        <state_interface name="position">
+          <param name="initial_value">0.0</param>
+        </state_interface>
+        <state_interface name="velocity"/>
+      </joint>
+  </ros2_control>
 </robot>
